File: hardware/NIMH-battery-charger.kicad_sch (KiCad schematic)
At the start: 44 parts, among them J1 Conn_01x03_Pin, J3 Conn_01x01_Pin, J4 Conn_01x01_Pin, J5 Conn_01x01_Pin, J6 Conn_01x01_Pin, J7 USB_C_Receptacle_PowerOnly_6P, U1 CH32V003f4u6

Commit message: Added comments on LED placement on PCB
Changed nanoCH32V003 code to print ADC immediately after start
Other:
- note added: "D7 is the main LED D5 - Bat 1 D6 - Bat 2 D8 - Bat 3 D10 - Bat 4"
Changed lines of the file:
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@@
+		)
+	)
+	(text "D7 is the main LED\nD5 - Bat 1\nD6 - Bat 2\nD8 - Bat 3\nD10 - Bat 4"
+		(exclude_from_sim no)
+		(at 214.376 24.892 0)
+		(effects
+			(font
+				(size 1.524 1.524)
+				(thickness 0.3048)
+				(bold yes)
+				(color 255 0 0 1)
+			)
+			(justify left)
 		)
 	)

Commit message: Add separte folders for main and devboard code
Add comments to hardware
Other:
- note added: "100R - ID30 1N4148 - ID162"
- note added: "Reverse LED - ID27 220R - ID94"
Changed lines of the file:
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@@
+		)
+	)
+	(text "100R - ID30\n1N4148 - ID162"
+		(exclude_from_sim no)
+		(at 225.044 95.758 0)
+		(effects
+			(font
+				(size 1.27 1.27)
+			)
+			(justify left)
+		)
+	)
+	(text "Reverse LED - ID27\n220R - ID94"
+		(exclude_from_sim no)
+		(at 174.752 18.034 0)
+		(effects
+			(font
+				(size 1.27 1.27)
+			)
+			(justify left)
 		)
 	)

Commit message: Adding comment to change the resistors
Other:
- note added: "Charging now with ~50mA Change R1 to R5 to 220 to reduce the charging current Charging current should be 20-30mA"
Changed lines of the file:
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@@
+		)
+	)
+	(text "Charging now with ~50mA\nChange R1 to R5 to 220 to reduce the charging current\nCharging current should be 20-30mA"
+		(exclude_from_sim no)
+		(at 238.252 101.854 0)
+		(effects
+			(font
+				(size 1.524 1.524)
+				(thickness 0.3048)
+				(bold yes)
+				(color 255 0 0 1)
+			)
 		)
 	)

Commit message: Add comments on measured charging current
Other:
- note added: "Measured charging current is 27 mA"
- note removed: "Charging now with ~50mA Change R1 to R5 to 220 to reduce the charging current Charging current should be 20-30mA"
Changed lines of the file:
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@@
 		)
 	)
-	(text "Charging now with ~50mA\nChange R1 to R5 to 220 to reduce the charging current\nCharging current should be 20-30mA"
+	(text "Measured charging current is 27 mA"
 		(exclude_from_sim no)
 		(at 238.252 101.854 0)
